Commit message: Upgraded camera sensor to Kinect RGB-D camera sensor

File: src/my_robot/urdf/my_robot.xacro (robot description, xacro)
@@ -147,4 +147,7 @@
     </visual>
   </link>
+  <!--New Camera link-->
+  <link name="camera_link_optical">
+  </link>
   <!--Hoyuko sensor link-->
   <link name="hokuyo">
@@ -215,3 +218,8 @@
     <axis xyz="0 1 0" rpy="0 0 0"/>
   </joint>
+  <joint name="camera_optical_joint" type="fixed">
+    <origin xyz="0 0 0" rpy="-1.5707 0 -1.5707"/>
+    <parent link="camera_link"/>
+    <child link="camera_link_optical"/>
+  </joint>
 </robot>

Commit message: Corrected parent link name in camera_optical_joint from camera_link to camera

File: src/my_robot/urdf/my_robot.xacro (robot description, xacro)
@@ -220,5 +220,5 @@
   <joint name="camera_optical_joint" type="fixed">
     <origin xyz="0 0 0" rpy="-1.5707 0 -1.5707"/>
-    <parent link="camera_link"/>
+    <parent link="camera"/>
     <child link="camera_link_optical"/>
   </joint>

Commit message: changed the reference name in my_robot.gazebo file from non-existent camera_link to existent camera_link optical

File: src/my_robot/urdf/my_robot.xacro (robot description, xacro)
@@ -219,5 +219,5 @@
   </joint>
   <joint name="camera_optical_joint" type="fixed">
-    <origin xyz="0 0 0" rpy="-1.5707 0 -1.5707"/>
+    <origin xyz="0 0 0" rpy="0 0 0"/>
     <parent link="camera"/>
     <child link="camera_link_optical"/>
